Commit message: PR06 realization

File: src/course_description/urdf/vehicle.urdf.xacro (robot description, xacro)
@@ -54,5 +54,5 @@
   </link>
   <joint name="lidar_joint" type="fixed">
-    <parent link="camera_link"/>
+    <parent link="base_link"/>
     <child link="lidar_link"/>
     <origin xyz="${wheelbase/2 - 0.05} 0 ${base_height/2 + lidar_height/2}" rpy="0 0 0"/>
